File: _restore_backup_2026-09-05T21-45-12-539/spotweldermainboard.kicad_pcb (KiCad board)
At the start: 2 copper layers, 80 x 150 mm, 50 parts, among them J1 tft_screen, J2 program, J3 Conn_01x02_Pin, J4 Conn_01x02_Pin, J5 MOT, J6 Conn_01x02_Pin, M1 Motor_DC, M2 Motor_DC, Q1 BC517, Q2 PN2222A, Q3 2N7000, Q4 2N7000, SW1 SW_Push, U1 CH32V003FxPx, U2 MOC3052M, U3 4N35, U4 BTA40-600B

Commit message: doing some wiring work, mcu is kinda hard to wire
Parts:
- D6, D8, U1: moved to B.Cu
- moved J4 32.6 mm to (106.5, 160.2), turned to 180 degrees
- moved R8 21.0 mm to (128.8, 89.3), turned to 90 degrees
- moved Q4 19.3 mm to (91.5, 146.5), turned to 180 degrees
- moved D10 16.8 mm to (96.8, 152.5), turned to 180 degrees
- moved U1 12.6 mm to (106.0, 108.5), turned to 0 degrees
- moved SW1 11.9 mm to (105.5, 117.0), turned to 0 degrees
- moved R2 11.5 mm to (118.4, 125.2), turned to -90 degrees
- moved D9 11.3 mm to (83.4, 152.7)
- moved M1 11.3 mm to (82.0, 160.2)
- moved M2 11.3 mm to (95.0, 160.2)
- moved R11 11.3 mm to (83.0, 140.4)
- moved R1 11.2 mm to (109.0, 137.7), turned to -90 degrees
- moved D6 10.3 mm to (115.3, 81.0), turned to 180 degrees
- moved Q3 8.58 mm to (78.3, 147.5), turned to 180 degrees
- moved D8 7.95 mm to (107.2, 95.5), turned to 0 degrees
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Connections:
- SW1 pad 1: ko -> Net-(U1-PD7)
- U1 pad 4: ko -> Net-(U1-PD7)
Routing:
- net blk: track 167.4 -> 0.00 mm
- net Ac1: track 95.3 -> 0.00 mm
- net gnd: track 56.9 -> 0.00 mm
- net trA: track 48.7 -> 0.00 mm
- net Net-(U2-Pad4): track 40.2 -> 0.00 mm
- net Net-(D10-A): track 36.7 -> 0.00 mm
- net Net-(D3-A): track 34.8 -> 0.00 mm
- net TriacB: track 34.1 -> 0.00 mm
- net +12V: track 33.4 -> 0.00 mm
- net Ac2: track 33.1 -> 0.00 mm
- net Net-(D1-A): track 30.3 -> 0.00 mm
- net Net-(R7-Pad1): track 24.3 -> 0.00 mm
- net psh: track 24.1 -> 0.00 mm
- net Out_crosszeroo: track 23.2 -> 0.00 mm
- net trB: track 19.8 -> 0.00 mm
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