File: _restore_backup_2026-09-05T21-45-12-539/spotweldermainboard.kicad_sch (KiCad schematic)
At the start: 50 parts, among them J1 tft_screen, J2 program, J3 Conn_01x02_Pin, J4 Conn_01x02_Pin, J5 MOT, J6 Conn_01x02_Pin, M1 Motor_DC, M2 Motor_DC, Q1 BC517, Q2 PN2222A, Q3 2N7000, Q4 2N7000, SW1 SW_Push, U1 CH32V003FxPx, U2 MOC3052M, U3 4N35, U4 BTA40-600B

Commit message: doing some wiring work, mcu is kinda hard to wire
Connections:
- net ko: no longer SW1.1, U1.4 (PD7)
- new net: SW1.1, U1.4 (PD7)
Changed lines of the file:
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@@
-	)
-	(junction
-		(at 68.58 49.53)
-		(diameter 0)
-		(color 0 0 0 0)
 	)
 	(junction
@@
 	(wire
 		(pts
-			(xy 71.12 49.53) (xy 68.58 49.53)
+			(xy 71.12 49.53) (xy 59.69 49.53)
 		)
 		(stroke
@@
 	(wire
 		(pts
-			(xy 68.58 49.53) (xy 59.69 49.53)
-		)
-		(stroke
-			(width 0)
-			(type default)
-		)
-	)
-	(wire
-		(pts
 			(xy 58.42 193.04) (xy 72.39 193.04)
 		)
@@
 		(pts
 			(xy 38.1 44.45) (xy 39.37 44.45)
-		)
-		(stroke
-			(width 0)
-			(type default)
-		)
-	)
-	(wire
-		(pts
-			(xy 68.58 53.34) (xy 68.58 49.53)
 		)
 		(stroke
@@
 			)
 		)
-	)
-	(global_label "ko"
-		(shape input)
-		(at 68.58 53.34 270)
-		(fields_autoplaced yes)
-		(effects
-			(font
-				(size 1.27 1.27)
-			)
-			(justify right)
-		)
-		(property "Intersheetrefs" "${INTERSHEET_REFS}"
-			(at 68.58 58.5023 90)
-			(hide yes)
-			(show_name no)
-			(do_not_autoplace no)
-			(effects
-				(font
-					(size 1.27 1.27)
-				)
-				(justify right)
-			)
-		)
