File: _restore_backup_2026-10-04T23-01-08-928/spotweldermainboard.kicad_pcb (KiCad board)
At the start: 2 copper layers, 80 x 150 mm, 50 parts, among them J1 tft_screen, J2 program, J3 Conn_01x02_Pin, J4 Conn_01x02_Pin, J5 MOT, J6 Conn_01x02_Pin, M1 Motor_DC, M2 Motor_DC, Q1 BC517, Q2 PN2222A, Q3 2N7000, Q4 2N7000, SW1 SW_Push, U1 CH32V003FxPx, U2 MOC3052M, U3 4N35, U4 BTA40-600B

Commit message: doing some wiring work, mcu is kinda hard to wire
Parts:
- D6, D8: moved to B.Cu
- moved D8 3.86 mm to (104.4, 89.8), turned to 0 degrees
- turned D6 to -90 degrees
Routing:
- net blk: track 167.4 -> 64.4 mm
- net gnd: track 56.9 -> 0.00 mm
- net trA: track 48.7 -> 0.00 mm
- net psh: track 24.1 -> 0.00 mm
- net res: track 17.3 -> 0.00 mm
- net sda: track 15.8 -> 0.00 mm
- net buzz: track 12.2 -> 0.00 mm
- net Net-(D6-A): track 6.16 -> 0.00 mm
- net Net-(J2-Pin_1): track 2.85 -> 0.00 mm
- net Net-(D8-A): track 2.49 -> 0.00 mm
- net Net-(R7-Pad1): track 24.3 -> 22.8 mm
- net mod: track 1.04 -> 0.00 mm
